File: open.kicad_pcb (KiCad board)
At the start: 2 copper layers, 64.1 x 40.5 mm, 9 parts, among them J1 BERG STRIP, J2 BERG STRIP

Commit message: made
Parts:
- moved J2 44.4 mm to (150.8, 86.9)
- moved U1 27.4 mm to (128.4, 98.7)
Changed lines of the file:
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@@
 	(footprint "Connector_PinSocket_2.00mm:PinSocket_1x04_P2.00mm_Vertical"
 		(layer "F.Cu")
-		(at 113.78 111.44)
+		(at 150.84 86.94)
 		(descr "Through hole straight socket strip, 1x04, 2.00mm pitch, single row (from Kicad 4.0.7), script generated")
 		(tags "Through hole socket strip THT 1x04 2.00mm single row")
@@
 	(footprint "EasyEDA:WIFI-SMD_ESP32-WROOM-32E"
 		(layer "F.Cu")
-		(at 155.85 98.65)
+		(at 128.445 98.65)
 		(property "Reference" "U1"
 			(at 0 -13 0)

Commit message: fdcdcdcdcd
Parts:
- moved J2 8.44 mm to (156.8, 92.9)
Changed lines of the file:
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@@
 	(footprint "Connector_PinSocket_2.00mm:PinSocket_1x04_P2.00mm_Vertical"
 		(layer "F.Cu")
-		(at 150.84 86.94)
+		(at 156.81 92.91)
 		(descr "Through hole straight socket strip, 1x04, 2.00mm pitch, single row (from Kicad 4.0.7), script generated")
 		(tags "Through hole socket strip THT 1x04 2.00mm single row")
